Commit message: add tiny hole model -2

File: robots/hydrus/urdf/hole.urdf (robot description, URDF)
Before this commit: robot hole, 1 links, 0 joints
Links:
- removed link base_link
- added link hole_link, mass 17.475; collision mesh filename=package://hydrus/urdf/mesh/scene/hole_link.dae; visual mesh filename=package://hydrus/urdf/mesh/scene/hole_link.dae

Commit message: add tiny hole model -3

File: robots/hydrus/urdf/hole.urdf (robot description, URDF)
Before this commit: robot hole, 1 links, 0 joints
Links:
- link hole_link: mass 17.475 -> 11.1367786842339
