Commit message: Update impedance_control
Now impedance control can be used in mini_quadrotor and hydyus
1. Support mode change, pub "{robot_name}/imp_rotor" to change mode. 0 for joint angle mode and 1 for position control mode, default is joint mode
2.Pub "{robot_name}/joint_cmds" to control joints in joint angle mode. Recommend value:pos[0.0, 0.785, 0.785] for mini_quadrotor, pos[1.26, 1.26, 1.26] for hydrus
3.Pub "{robot_name}/pos_cmds" to control end_effector's position in position control mode. Recommend value:[x:0.0, y:0.1, z:-0.2] for mini_quadrotor, pos[x:-0.6, y:0.2, z:0.0] for hydrus

File: robots/hydrus/urdf/common.xacro (robot description, xacro)
@@ -126,4 +126,19 @@
     </xacro:extra_module>
   </xacro:macro>
+  <joint name="joint_eff" type="fixed">
+      <parent link="link4"/>
+      <child link="end_effector"/>
+      <origin rpy="0 0 0" xyz="${link_length} 0 0"/>
+    </joint>
+    <link name="end_effector">
+     <inertial>
+        <origin xyz="0 0 0" rpy="0 0 0"/>
+        <mass value="0.001"/>
+        <inertia
+            ixx="0.0001" ixy="0.0" ixz="0.0"
+            iyy="0.0001" iyz="0.0"
+            izz="0.0001"/>
+      </inertial>
+    </link>
   <!-- friction -->
   <xacro:macro name="friction" params="self">

Commit message: merge to main PC

File: robots/hydrus/urdf/common.xacro (robot description, xacro)
@@ -130,15 +130,51 @@
       <child link="end_effector"/>
       <origin rpy="0 0 0" xyz="${link_length} 0 0"/>
-    </joint>
-    <link name="end_effector">
-     <inertial>
-        <origin xyz="0 0 0" rpy="0 0 0"/>
-        <mass value="0.001"/>
-        <inertia
-            ixx="0.0001" ixy="0.0" ixz="0.0"
-            iyy="0.0001" iyz="0.0"
-            izz="0.0001"/>
-      </inertial>
-    </link>
+  </joint>
+  <link name="end_effector">
+    <inertial>
+      <origin xyz="0 0 0" rpy="0 0 0"/>
+      <mass value="0.001"/>
+      <inertia
+          ixx="0.0001" ixy="0.0" ixz="0.0"
+          iyy="0.0001" iyz="0.0"
+          izz="0.0001"/>
+    </inertial>
+      <collision>
+        <origin rpy="0 0 0" xyz="0 0 0"/>
+        <geometry>
+          <sphere radius="0.02"/>
+        </geometry>
+      </collision>
+      <visual>
+        <origin rpy="0 0 0" xyz="0 0 0"/>
+        <geometry>
+          <sphere radius="0.02"/>
+        </geometry>
+      </visual>
+  </link>
+  <gazebo reference="end_effector">
+    <sensor name="contacts" type="contact">
+        <contact>
+          <collision>link4_fixed_joint_lump__end_effector_collision_1</collision>
+        </contact>
+        <plugin name="gazebo_ros_bumper_controller" filename="libgazebo_ros_bumper.so">
+          <always_on>true</always_on>
+          <robotNamespace>/hydrus</robotNamespace>
+          <bumperTopicName>bumper_states</bumperTopicName>
+          <frameName>bumper</frameName>
+          <visualize>true</visualize>
+          <update_rate>1000.0</update_rate>
+        </plugin>
+    </sensor>
+  </gazebo>
+  <!-- <gazebo>
+    <plugin name="contact_plugin" filename="libgazebo_ros_contact.so">
+      <ros>
+        <namespace>/contact_test</namespace>
+        <remapping>contact_topic:=contact_states</remapping>
+      </ros>
+      <collisionName>link4_fixed_joint_lump__end_effector_collision_1</collisionName>
+    </plugin>
+  </gazebo> -->
   <!-- friction -->
   <xacro:macro name="friction" params="self">

Commit message: test commit in new PC -1

File: robots/hydrus/urdf/common.xacro (robot description, xacro)
@@ -126,4 +126,55 @@
     </xacro:extra_module>
   </xacro:macro>
+  <joint name="joint_eff" type="fixed">
+      <parent link="link4"/>
+      <child link="end_effector"/>
+      <origin rpy="0 0 0" xyz="${link_length} 0 0"/>
+  </joint>
+  <link name="end_effector">
+    <inertial>
+      <origin xyz="0 0 0" rpy="0 0 0"/>
+      <mass value="0.001"/>
+      <inertia
+          ixx="0.0001" ixy="0.0" ixz="0.0"
+          iyy="0.0001" iyz="0.0"
+          izz="0.0001"/>
+    </inertial>
+      <collision>
+        <origin rpy="0 0 0" xyz="0 0 0"/>
+        <geometry>
+          <sphere radius="0.02"/>
+        </geometry>
+      </collision>
+      <visual>
+        <origin rpy="0 0 0" xyz="0 0 0"/>
+        <geometry>
+          <sphere radius="0.02"/>
+        </geometry>
+      </visual>
+  </link>
+  <gazebo reference="end_effector">
+    <sensor name="contacts" type="contact">
+        <contact>
+          <collision>link4_fixed_joint_lump__end_effector_collision_1</collision>
+        </contact>
+        <plugin name="gazebo_ros_bumper_controller" filename="libgazebo_ros_bumper.so">
+          <always_on>true</always_on>
+          <robotNamespace>/hydrus</robotNamespace>
+          <bumperTopicName>bumper_states</bumperTopicName>
+          <frameName>bumper</frameName>
+          <visualize>true</visualize>
+          <update_rate>1000.0</update_rate>
+        </plugin>
+    </sensor>
+  </gazebo>
+  <!-- <gazebo>
+    <plugin name="contact_plugin" filename="libgazebo_ros_contact.so">
+      <ros>
+        <namespace>/contact_test</namespace>
+        <remapping>contact_topic:=contact_states</remapping>
+      </ros>
+      <collisionName>link4_fixed_joint_lump__end_effector_collision_1</collisionName>
+    </plugin>
+  </gazebo> -->
   <!-- friction -->
   <xacro:macro name="friction" params="self">

Commit message: add tiny hole model -4

File: robots/hydrus/urdf/common.xacro (robot description, xacro)
@@ -131,4 +131,5 @@
       <origin rpy="0 0 0" xyz="${link_length} 0 0"/>
   </joint>
+<!--
   <link name="end_effector">
     <inertial>
@@ -150,4 +151,26 @@
         <geometry>
           <sphere radius="0.02"/>
+        </geometry>
+      </visual>
+  </link> -->
+  <link name="end_effector">
+    <inertial>
+      <origin xyz="0 0 0" rpy="0 0 1.57"/>
+      <mass value="0.001"/>
+      <inertia
+          ixx="0.0001" ixy="0.0" ixz="0.0"
+          iyy="0.0001" iyz="0.0"
+          izz="0.0001"/>
+    </inertial>
+      <collision>
+        <origin rpy="0 1.57 0" xyz="0.3 0 0"/>
+        <geometry>
+          <cylinder length="0.6" radius="0.01"/>
+        </geometry>
+      </collision>
+      <visual>
+        <origin rpy="0 1.57 0" xyz="0.3 0 0"/>
+        <geometry>
+          <cylinder length="0.6" radius="0.01"/>
         </geometry>
       </visual>

Commit message: store the current modification

File: robots/hydrus/urdf/common.xacro (robot description, xacro)
@@ -131,5 +131,4 @@
       <origin rpy="0 0 0" xyz="${link_length} 0 0"/>
   </joint>
-<!--
   <link name="end_effector">
     <inertial>
@@ -153,5 +152,6 @@
         </geometry>
       </visual>
-  </link> -->
+  </link>
+<!--
   <link name="end_effector">
     <inertial>
@@ -175,5 +175,5 @@
         </geometry>
       </visual>
-  </link>
+  </link> -->
   <gazebo reference="end_effector">
     <sensor name="contacts" type="contact">

File: robots/hydrus_xi/urdf/common.xacro (robot description, xacro)
@@ -44,4 +44,26 @@
       <origin rpy="0 0 0" xyz="${link_length} 0 0"/>
   </joint>
+  <!-- <link name="end_effector">
+    <inertial>
+      <origin xyz="0 0 0" rpy="0 0 0"/>
+      <mass value="0.001"/>
+      <inertia
+          ixx="0.0001" ixy="0.0" ixz="0.0"
+          iyy="0.0001" iyz="0.0"
+          izz="0.0001"/>
+    </inertial>
+      <collision>
+        <origin rpy="0 0 0" xyz="0 0 0"/>
+        <geometry>
+          <sphere radius="0.02"/>
+        </geometry>
+      </collision>
+      <visual>
+        <origin rpy="0 0 0" xyz="0 0 0"/>
+        <geometry>
+          <sphere radius="0.02"/>
+        </geometry>
+      </visual>
+  </link>  -->
   <link name="end_effector">
     <inertial>

File: robots/hydrus_xi/urdf/hole.urdf (robot description, URDF)
Before this commit: robot hole, 1 links, 0 joints
Links:
- link hole_link: geometry collision mesh filename=package://hydrus/urdf/mesh/scene/wall_link.dae; visual mesh filename=package://hydrus/urdf/mesh/scene/wall_link.dae
