Commit message: change to hudrus_xi

File: robots/hydrus_xi/urdf/common.xacro (robot description, xacro)
@@ -39,4 +39,46 @@
     </collision>
   </xacro:macro>
+    <joint name="joint_eff" type="fixed">
+      <parent link="link4"/>
+      <child link="end_effector"/>
+      <origin rpy="0 0 0" xyz="${link_length} 0 0"/>
+  </joint>
+  <link name="end_effector">
+    <inertial>
+      <origin xyz="0 0 0" rpy="0 0 1.57"/>
+      <mass value="0.001"/>
+      <inertia
+          ixx="0.0001" ixy="0.0" ixz="0.0"
+          iyy="0.0001" iyz="0.0"
+          izz="0.0001"/>
+    </inertial>
+      <collision>
+        <origin rpy="0 1.57 0" xyz="0.3 0 0"/>
+        <geometry>
+          <cylinder length="0.6" radius="0.01"/>
+        </geometry>
+      </collision>
+      <visual>
+        <origin rpy="0 1.57 0" xyz="0.3 0 0"/>
+        <geometry>
+          <cylinder length="0.6" radius="0.01"/>
+        </geometry>
+      </visual>
+  </link>
+  <gazebo reference="end_effector">
+    <sensor name="contacts" type="contact">
+        <contact>
+          <collision>link4_fixed_joint_lump__end_effector_collision_1</collision>
+        </contact>
+        <plugin name="gazebo_ros_bumper_controller" filename="libgazebo_ros_bumper.so">
+          <always_on>true</always_on>
+          <robotNamespace>/hydrus</robotNamespace>
+          <bumperTopicName>bumper_states</bumperTopicName>
+          <frameName>bumper</frameName>
+          <visualize>true</visualize>
+          <update_rate>1000.0</update_rate>
+        </plugin>
+    </sensor>
+  </gazebo>
   <xacro:macro name="extra_module" params="name parent *origin *inertial visible:=0 model_url:=0">
     <joint name="${parent}2${name}" type="fixed">
