Commit message: update

File: robots/hydrus_xi/urdf/hole.urdf (robot description, URDF)
Before this commit: robot hole, 1 links, 0 joints
Links:
- link hole_link: geometry collision mesh filename=package://hydrus/urdf/mesh/scene/hole_link.dae; visual mesh filename=package://hydrus/urdf/mesh/scene/hole_link.dae
